File: unmechanical-sweepish/unmechanical-sweepish.kicad_pcb (KiCad board)
At the start: 4 copper layers, 214 x 145.5 mm, 168 parts, among them J1 HytePro M, J2 USB_C_Receptacle_USB2.0, J3 M, J4 HytePro F, J5 USB_C_Receptacle_USB2.0, J6 M, Q1 AO3400A, Q2 AO3400A, SW1 B/R, SW2 B/R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

Commit message: Rotate halves together
Parts:
- moved H6 242.4 mm to (270.4, 81.4), turned to 2 degrees
- moved J1 238.5 mm to (147.4, 92.1), turned to 88 degrees
- moved EC33 235.6 mm to (259.6, 94.4), turned to 16 degrees
- moved R2 234.7 mm to (144.4, 88.1), turned to -2 degrees
- moved R41 234.5 mm to (244.1, 115.2), turned to 16 degrees
- moved R1 234.2 mm to (144.4, 89.3), turned to -2 degrees
- moved H2 232.5 mm to (131.2, 54.3), turned to -2 degrees
- moved H3 232.3 mm to (144.6, 133.3), turned to -2 degrees
- moved R40 231.9 mm to (243.6, 113.5), turned to 16 degrees
- moved C35 231.2 mm to (240.6, 116.4), turned to -164 degrees
- moved JP1 230.3 mm to (143.5, 97.9), turned to 178 degrees
- moved R3 229.7 mm to (143.4, 100.1), turned to -2 degrees
- moved J3 229.4 mm to (143.5, 102.9), turned to 88 degrees
- moved R39 229.3 mm to (243.1, 111.8), turned to 16 degrees
- moved R42 226.7 mm to (242.6, 110.1), turned to 16 degrees
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Other:
- board size 214 x 145.5 mm -> 252.8 x 128.9 mm
- board text removed: "UnMechanical Sweepish by ebastler Capacitive touch-keyboard, rev0.1"

Commit message: Fix up for order
Parts:
- J1: footprint PCM_marbastlib-xp-various:CON_HytePro_M411P_Plug_1x04-P2.20mm_Horizontal_FlushMount -> Connector_PinHeader_2.54mm:PinHeader_1x04_P2.54mm_Vertical; moved to F.Cu
- J4: footprint PCM_marbastlib-xp-various:CON_HytePro_M411P_Receptacle_1x04-P2.20mm_Horizontal_FlushMount -> Connector_PinHeader_2.54mm:PinHeader_1x04_P2.54mm_Vertical; moved to F.Cu
- L1, L2: value BLM15PX121SN1D -> BLM15PX121SN1D
- moved J4 10.3 mm to (158.0, 82.6), turned to 0 degrees
- moved J1 9.66 mm to (149.0, 82.6), turned to 0 degrees
Routing:
- net Net-(J4-Pin_2): track 2.75 -> 13.8 mm
- net Net-(J1-Pin_2): track 2.76 -> 10.7 mm
- net Net-(J4-Pin_3): track 2.75 -> 6.77 mm
- net Net-(J1-Pin_3): track 2.76 -> 4.25 mm
